File: eagle/mike_sims_vca.sch (EAGLE design)
At the start: 30 parts, among them IC2 LM13700N, IC3 TL072P, Q1 2N3906

Commit message: nearly routed
Parts:
- added GAIN: 100k, pot:3RP/1610N
- added R6: 20k, rcl:R-US_0207/10
- added R7: 100k, rcl:R-US_0207/10
Connections:
- new net N$12: GAIN.S, R6.2
- new net N$13: GAIN.E, R7.2
- net +12V: now also R7.1
- net GND: now also GAIN.A
- net N$20: now also R6.1
Changed lines of the file:
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@@
 <part name="C12" library="rcl" deviceset="C-US" device="050-024X044" value="390p"/>
 <part name="R5" library="rcl" deviceset="R-US_" device="0207/10" value="10k"/>
+<part name="GAIN" library="pot" deviceset="3RP/1610N" device="" value="100k"/>
+<part name="R6" library="rcl" deviceset="R-US_" device="0207/10" value="20k"/>
+<part name="P+2" library="supply1" deviceset="+12V" device=""/>
+<part name="R7" library="rcl" deviceset="R-US_" device="0207/10" value="100k"/>
+<part name="GND10" library="supply1" deviceset="GND" device=""/>
 </parts>
 <sheets>
@@
 <instance part="C12" gate="G$1" x="154.94" y="45.72" rot="R90"/>
 <instance part="R5" gate="G$1" x="137.16" y="33.02" rot="R180"/>
+<instance part="GAIN" gate="G$1" x="198.12" y="50.8" rot="MR0"/>
+<instance part="R6" gate="G$1" x="175.26" y="50.8"/>
+<instance part="P+2" gate="1" x="198.12" y="73.66"/>
+<instance part="R7" gate="G$1" x="198.12" y="63.5" rot="R270"/>
+<instance part="GND10" gate="1" x="198.12" y="40.64"/>
 </instances>
 <busses>
@@
 <pinref part="P+4" gate="1" pin="+12V"/>
 <wire x1="50.8" y1="78.74" x2="50.8" y2="76.2" width="0.1524" layer="91"/>
+</segment>
+<segment>
+<pinref part="P+2" gate="1" pin="+12V"/>
+<pinref part="R7" gate="G$1" pin="1"/>
+<wire x1="198.12" y1="68.58" x2="198.12" y2="71.12" width="0.1524" layer="91"/>
 </segment>
 </net>
@@
 <wire x1="162.56" y1="25.4" x2="162.56" y2="30.48" width="0.1524" layer="91"/>
 </segment>
+<segment>
+<pinref part="GAIN" gate="G$1" pin="A"/>
+<pinref part="GND10" gate="1" pin="GND"/>
+<wire x1="198.12" y1="43.18" x2="198.12" y2="45.72" width="0.1524" layer="91"/>
+</segment>
 </net>
 <net name="N$19" class="0">
@@
 <junction x="165.1" y="45.72"/>
 <pinref part="IC3" gate="B" pin="-IN"/>
+<pinref part="R6" gate="G$1" pin="1"/>
+<wire x1="165.1" y1="50.8" x2="170.18" y2="50.8" width="0.1524" layer="91"/>
+<junction x="165.1" y="50.8"/>
 </segment>
 </net>
@@
 </segment>
 </net>
+<net name="N$12" class="0">
+<segment>
+<pinref part="R6" gate="G$1" pin="2"/>
+<pinref part="GAIN" gate="G$1" pin="S"/>
+<wire x1="180.34" y1="50.8" x2="193.04" y2="50.8" width="0.1524" layer="91"/>
+</segment>
+</net>
+<net name="N$13" class="0">
+<segment>
+<pinref part="GAIN" gate="G$1" pin="E"/>
+<pinref part="R7" gate="G$1" pin="2"/>
+<wire x1="198.12" y1="58.42" x2="198.12" y2="55.88" width="0.1524" layer="91"/>
+</segment>
+</net>
